File: pcb/left/keyboard_pcb.kicad_sch (KiCad schematic)
At the start: 33 parts, among them J1 TRRS, K00 KEYSW, K01 KEYSW, K02 KEYSW, K03 KEYSW, K04 KEYSW, K05 KEYSW, K10 KEYSW, K11 KEYSW, K12 KEYSW, K13 KEYSW, K14 KEYSW, K15 KEYSW, K20 KEYSW, K21 KEYSW, K22 KEYSW, K23 KEYSW, K24 KEYSW, K25 KEYSW, K30 KEYSW, K31 KEYSW, K32 KEYSW, U2 Pico

Commit message: feat: update
Parts:
- added H5, H6, H7, H8: MountingHole, beekeeb_lib:MountingHole_2.2mm_M2-8mm, symbol Mechanical:MountingHole
- added J2: TRRS, Resistor_SMD:R_1206_3216Metric_Pad1.30x1.75mm_HandSolder, symbol keebio:TRRS
- added K16, K17, K18, K19, K26, K27, K28, K29, K33, K34, K35, K36, K37, K38, K39, K40, K41, K6, K7, K8, K9: KEYSW, keyswitches:SW_PG1350_reversible, symbol keyboard_parts:KEYSW
- added MB5, MB6, MB7, MB8: MountingHole, beekeeb_lib:mousebites, symbol Mechanical:MountingHole
- added R3: 5k6, Resistor_SMD:R_1206_3216Metric_Pad1.30x1.75mm_HandSolder, symbol Device:R
- added R4: 10k, Resistor_SMD:R_1206_3216Metric_Pad1.30x1.75mm_HandSolder, symbol Device:R
- added U1: Pico, RPi_Pico:RPi_Pico_SMD_TH, symbol KiCad-RP-Pico:Pico
Connections:
- net GND: now also J2.3 (RING1), K16.2, K17.2, K18.2, K19.2, K26.2, K27.2, K28.2, K29.2, K33.2, K34.2, K35.2, K36.2, K37.2, K38.2, K39.2, K40.2, K41.2, K6.2, K7.2, K8.2, K9.2, R4.2, U1.13 (GND), U1.18 (GND), U1.23 (GND), U1.28 (GND), U1.3 (GND), U1.33 (AGND), U1.38 (GND), U1.8 (GND)
- net VBUS: now also R3.1, U1.40 (VBUS)
- net VCC: now also J2.2 (TIP), U1.39 (VSYS)
- net k00: now also K6.1, U1.15 (GPIO11)
- net k01: now also K9.1, U1.11 (GPIO8)
- net k02: now also K18.1, U1.7 (GPIO5)
- net k03: now also K27.1, U1.4 (GPIO2)
- net k04: now also K34.1, U1.27 (GPIO21)
- net k05: now also K38.1, U1.29 (GPIO22)
- net k10: now also K7.1, U1.16 (GPIO12)
- net k11: now also K16.1, U1.12 (GPIO9)
- net k12: now also K19.1, U1.9 (GPIO6)
- net k13: now also K28.1, U1.5 (GPIO3)
- net k14: now also K35.1, U1.25 (GPIO19)
- net k15: now also K39.1, U1.26 (GPIO20)
- net k20: now also K8.1, U1.17 (GPIO13)
- net k21: now also K17.1, U1.14 (GPIO10)
- net k22: now also K26.1, U1.10 (GPIO7)
- net k23: now also K29.1, U1.6 (GPIO4)
- net k24: now also K36.1, U1.22 (GPIO17)
- net k25: now also K40.1, U1.24 (GPIO18)
- net k30: now also K33.1, U1.21 (GPIO16)
- net k31: now also K37.1, U1.19 (GPIO14)
- net k32: now also K41.1, U1.20 (GPIO15)
- net rx: now also J2.4 (RING2), U1.2 (GPIO1)
- net tx: now also J2.1 (SLEEVE), U1.1 (GPIO0)
- net vbus_sense: now also R3.2, R4.1, U1.34 (GPIO28_ADC2)
- no-connect marks 9 -> 18
Other:
- moved on the sheet: K00, K01, K02, K03, K04, K05, K10, K11, K12, K13, K14, K15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
